File: pcb/flipdot-brose.kicad_pcb (KiCad board)
At the start: 2 copper layers, 100 x 100 mm, 195 parts, among them J1 Conn_02x30_Odd_Even, J2 Conn_01x03, J3 Conn_01x02, J4 Conn_01x02, U1 ESP32_DEVCITV1, U10 ULN2803A, U11 ULN2803A, U12 74HC595, U13 TBD62783A, U14 74HC595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

Commit message: resistor/capacitor for leds
Parts:
- removed the REF** at (172.9, 83.7)
- removed the REF** at (174.4, 82.2)
- removed the REF** at (175.9, 82.2)
- removed the REF** at (175.9, 83.7)
- removed the REF** at (172.9, 80.7)
- removed the REF** at (177.4, 80.7)
- removed the REF** at (175.9, 80.7)
- removed the REF** at (177.4, 83.7)
- removed the REF** at (172.9, 82.2)
- removed the REF** at (177.4, 82.2)
- removed the REF** at (174.4, 80.7)
- removed the REF** at (174.4, 83.7)
- added C3: 1000u, Capacitor_THT:CP_Radial_D10.0mm_P5.00mm, F.Cu at (194.4, 99.4)
- added R11: 330, Resistor_THT:R_Axial_DIN0204_L3.6mm_D1.6mm_P5.08mm_Horizontal, F.Cu at (179.7, 106.2)
- moved D2 25.5 mm to (174.4, 84.7)
- moved R9 3.54 mm to (182.4, 80.7)
- moved R10 2.66 mm to (184.9, 82.5)
Connections:
- J2 pad 2: DATA-LED -> Net-(J2-Pad2)
Routing:
- net Net-(D2-Pad2): track 49.7 -> 77.0 mm, vias 0 -> 2
- net VCC-LED: track 46.4 -> 59.0 mm
- net Net-(J2-Pad2): track 0.00 -> 12.2 mm
- net DATA-LED: track 31.1 -> 23.5 mm, vias 1 -> 0
- net OE-SEL-3V3: track 57.5 -> 61.1 mm
- net SRCLR-3V3: track 48.2 -> 51.1 mm
- net OE-CONF-3V3: track 66.5 -> 69.1 mm
- net +3V3: track 59.9 -> 59.3 mm
